File: Electronics/frankShield.brd (EAGLE design)
At the start: 68.6 x 53.3 mm, 27 parts, among them IC1 BD6230F, IC2 BD6230F, IC3 TS5A23157

Commit message: Wemos MINI PCB added. Corrections to battery holder W.I.P.
Parts:
- removed LED1: (no value), led:CHIP-LED0805
- removed R4: 180R, rcl:M0805
Connections:
- removed net N$19: LED1.A, R4.2
- removed net N$20: R4.1, U$1.D9
- net GND: no longer LED1.C
- net N$17: now also U$1.D9; no longer U$1.D11
Routing:
- net N$20: track 12.5 -> 0.00 mm, vias 1 -> 0
- net N$19: track 3.08 -> 0.00 mm
- net N$17: track 58.3 -> 57.1 mm
Changed lines of the file:
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@@
 <?xml version="1.0" encoding="utf-8"?>
 <!DOCTYPE eagle SYSTEM "eagle.dtd">
-<eagle version="8.2.1">
+<eagle version="7.5.0">
 <drawing>
 <settings>
@@
 <element name="C7" library="rcl" package="C0805" value="0.1uF" x="19.3675" y="23.1775" rot="R180"/>
 <element name="D1" library="diode" package="SOD323_ST" value="BAT60J" x="59.3725" y="11.43"/>
-<element name="LED1" library="led" package="CHIP-LED0805" value="" x="23.1775" y="47.9425" rot="R90"/>
-<element name="R4" library="rcl" package="M0805" value="180R" x="28.2575" y="47.9425" rot="R180"/>
 </elements>
 <signals>
@@
 <contactref element="C6" pad="2"/>
 <contactref element="C7" pad="2"/>
-<contactref element="LED1" pad="C"/>
+<wire x1="42.5425" y1="31.4325" x2="53.975" y2="43.815" width="0" layer="19" extent="1-1"/>
+<wire x1="40.64" y1="23.495" x2="42.5425" y2="31.4325" width="0" layer="19" extent="1-1"/>
+<wire x1="40.955" y1="19.05" x2="40.955" y2="21.59" width="0" layer="19" extent="1-1"/>
+<wire x1="41.275" y1="13.97" x2="40.955" y2="19.05" width="0" layer="19" extent="1-1"/>
+<wire x1="33.02" y1="26.67" x2="38.1" y2="24.5569" width="0" layer="19" extent="1-1"/>
+<wire x1="40.64" y1="2.54" x2="41.275" y2="13.97" width="0" layer="19" extent="1-1"/>
+<wire x1="43.18" y1="2.54" x2="40.64" y2="2.54" width="0" layer="19" extent="1-1"/>
+<wire x1="55.88" y1="8.89" x2="43.18" y2="2.54" width="0" layer="19" extent="1-1"/>
+<wire x1="63.1825" y1="8.89" x2="55.88" y2="8.89" width="0" layer="19" extent="1-1"/>
+<wire x1="18.4175" y1="23.1775" x2="33.02" y2="26.67" width="0" layer="19" extent="1-1"/>
+<wire x1="18.415" y1="20.38" x2="18.4175" y2="23.1775" width="0" layer="19" extent="1-1"/>
+<wire x1="18.735" y1="32.385" x2="18.4175" y2="23.1775" width="0" layer="19" extent="1-1"/>
+<wire x1="18.415" y1="40.7" x2="18.735" y2="32.385" width="0" layer="19" extent="1-1"/>
+<wire x1="17.78" y1="46.355" x2="18.415" y2="40.7" width="0" layer="19" extent="1-1"/>
+<wire x1="26.416" y1="50.8" x2="17.78" y2="46.355" width="0" layer="19" extent="1-1"/>
+<wire x1="17.78" y1="6.985" x2="18.415" y2="20.38" width="0" layer="19" extent="1-1"/>
+<wire x1="3.81" y1="11.43" x2="17.78" y2="6.985" width="0" layer="19" extent="1-1"/>
 </signal>
 <signal name="VIN">
@@
 <wire x1="26.9875" y1="10.16" x2="27.6225" y2="10.795" width="0.8128" layer="16"/>
 <wire x1="27.6225" y1="36.83" x2="27.6225" y2="10.795" width="0.8128" layer="16"/>
-<contactref element="U$1" pad="D11"/>
 <wire x1="33.02" y1="42.2275" x2="27.6225" y2="36.83" width="0.8128" layer="16"/>
-<wire x1="34.036" y1="50.8" x2="34.036" y2="49.5935" width="0.8128" layer="16"/>
 <wire x1="34.036" y1="49.5935" x2="33.02" y2="48.5775" width="0.8128" layer="16"/>
 <wire x1="33.02" y1="48.5775" x2="33.02" y2="42.2275" width="0.8128" layer="16"/>
+<contactref element="U$1" pad="D9"/>
+<wire x1="34.036" y1="49.5935" x2="39.116" y2="50.8" width="0" layer="19" extent="16-16"/>
 </signal>
 <signal name="N$18">
@@
 <wire x1="61.595" y1="11.43" x2="60.6225" y2="11.43" width="0.8128" layer="1"/>
 </signal>
-<signal name="N$19">
-<contactref element="R4" pad="2"/>
-<contactref element="LED1" pad="A"/>
-<wire x1="27.3075" y1="47.9425" x2="24.2275" y2="47.9425" width="0.8128" layer="1"/>
-</signal>
-<signal name="N$20">
-<contactref element="U$1" pad="D9"/>
-<contactref element="R4" pad="1"/>
-<wire x1="39.116" y1="50.8" x2="39.116" y2="48.3235" width="0.8128" layer="16"/>
-<wire x1="39.116" y1="48.3235" x2="38.735" y2="47.9425" width="0.8128" layer="16"/>
-<wire x1="38.735" y1="47.9425" x2="34.925" y2="47.9425" width="0.8128" layer="16"/>
-<via x="34.925" y="47.9425" extent="1-16" drill="0.35"/>
-<wire x1="29.2075" y1="47.9425" x2="34.925" y2="47.9425" width="0.8128" layer="1"/>
-</signal>
 </signals>
