File: Electronics/frankShield.sch (EAGLE design)
At the start: 27 parts, among them IC1 BD6230F, IC2 BD6230F, IC3 TS5A23157

Commit message: PCB test program updated; all works.
TODO: write motor callibration function
      update schematic and PCB to take account of the use of the
      LED pin for input
Other:
- note added: "no connect"
Changed lines of the file:
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@@
 <text x="90.17" y="74.93" size="1.778" layer="96" rot="R90">batt volts</text>
 <text x="-78.74" y="114.3" size="1.778" layer="95">Note: wheel sensors take too much current to run off 3v3.</text>
+<wire x1="35.56" y1="66.04" x2="35.56" y2="63.5" width="0.1524" layer="95"/>
+<wire x1="35.56" y1="63.5" x2="33.02" y2="63.5" width="0.1524" layer="95"/>
+<wire x1="33.02" y1="63.5" x2="30.48" y2="63.5" width="0.1524" layer="95"/>
+<wire x1="30.48" y1="63.5" x2="30.48" y2="66.04" width="0.1524" layer="95"/>
+<wire x1="33.02" y1="63.5" x2="33.02" y2="66.04" width="0.1524" layer="95"/>
+<text x="27.94" y="60.96" size="1.778" layer="95">no connect</text>
 </plain>
 <instances>

Commit message: Wemos MINI PCB added. Corrections to battery holder W.I.P.
Parts:
- removed LED1: (no value), led:LEDCHIP-LED0805
- removed R4: 180R, rcl:R-EU_M0805
Connections:
- removed net N$19: LED1.A, R4.2
- removed net N$20: R4.1, U$1.D9
- net GND: no longer LED1.C
- net N$17: now also U$1.D9; no longer U$1.D11
Changed lines of the file:
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@@
 <?xml version="1.0" encoding="utf-8"?>
 <!DOCTYPE eagle SYSTEM "eagle.dtd">
-<eagle version="8.2.1">
+<eagle version="7.5.0">
 <drawing>
 <settings>
@@
 <part name="P+5" library="supply1" deviceset="V+" device="" value="+6V5"/>
 <part name="D1" library="diode" deviceset="BAT60J" device=""/>
-<part name="LED1" library="led" deviceset="LED" device="CHIP-LED0805"/>
-<part name="GND11" library="supply1" deviceset="GND" device=""/>
-<part name="R4" library="rcl" deviceset="R-EU_" device="M0805" value="180R"/>
 </parts>
 <sheets>
@@
 <instance part="P+5" gate="1" x="-45.72" y="109.22"/>
 <instance part="D1" gate="G$1" x="-63.5" y="71.12"/>
-<instance part="LED1" gate="G$1" x="20.32" y="104.14" rot="R270"/>
-<instance part="GND11" gate="1" x="12.7" y="99.06" rot="MR0"/>
-<instance part="R4" gate="G$1" x="30.48" y="104.14" rot="R180"/>
 </instances>
 <busses>
@@
 <wire x1="38.1" y1="127" x2="43.18" y2="127" width="0.1524" layer="91"/>
 </segment>
-<segment>
-<pinref part="LED1" gate="G$1" pin="C"/>
-<pinref part="GND11" gate="1" pin="GND"/>
-<wire x1="15.24" y1="104.14" x2="12.7" y2="104.14" width="0.1524" layer="91"/>
-<wire x1="12.7" y1="104.14" x2="12.7" y2="101.6" width="0.1524" layer="91"/>
-</segment>
 </net>
 <net name="+3V3" class="0">
@@
 <segment>
 <pinref part="JP9" gate="A" pin="2"/>
-<wire x1="35.56" y1="91.44" x2="-17.78" y2="91.44" width="0.1524" layer="91"/>
+<wire x1="40.64" y1="91.44" x2="-17.78" y2="91.44" width="0.1524" layer="91"/>
 <wire x1="-17.78" y1="91.44" x2="-17.78" y2="96.52" width="0.1524" layer="91"/>
-<pinref part="U$1" gate="G$1" pin="D11"/>
-<wire x1="35.56" y1="78.74" x2="35.56" y2="91.44" width="0.1524" layer="91"/>
+<pinref part="U$1" gate="G$1" pin="D9"/>
+<wire x1="40.64" y1="78.74" x2="40.64" y2="91.44" width="0.1524" layer="91"/>
 </segment>
 </net>
@@
 </segment>
 </net>
-<net name="N$19" class="0">
-<segment>
-<pinref part="R4" gate="G$1" pin="2"/>
-<pinref part="LED1" gate="G$1" pin="A"/>
-<wire x1="25.4" y1="104.14" x2="22.86" y2="104.14" width="0.1524" layer="91"/>
-</segment>
-</net>
-<net name="N$20" class="0">
-<segment>
-<pinref part="U$1" gate="G$1" pin="D9"/>
-<wire x1="40.64" y1="78.74" x2="40.64" y2="96.52" width="0.1524" layer="91"/>
-<wire x1="40.64" y1="96.52" x2="35.56" y2="96.52" width="0.1524" layer="91"/>
-<pinref part="R4" gate="G$1" pin="1"/>
-<wire x1="35.56" y1="96.52" x2="35.56" y2="104.14" width="0.1524" layer="91"/>
-</segment>
-</net>
