File: Frank 2.0/Electronics/Frank-2-Pi/Frank-2-Pi.sch (KiCad schematic (older format))
At the start: 11 parts, among them J2 Left motor, J3 Right motor, Q1 DMN6075S, Q2 DMN6075S, U1 adafruit-2448

Commit message: Frank 2 electronics WIP.
Parts:
- added C? (x6): 0.1u, Capacitor_SMD:C_0805_2012Metric, symbol Device:C_Small
- added C?: 10u, Capacitor_Tantalum_SMD:CP_EIA-3216-18_Kemet-A_Pad1.58x1.35mm_HandSolder, symbol Device:CP
- added C?: 100u, Capacitor_Tantalum_SMD:CP_EIA-3216-18_Kemet-A_Pad1.58x1.35mm_HandSolder, symbol Device:CP
- added J?: LIDAR, Connector_PinHeader_2.54mm:PinHeader_1x04_P2.54mm_Vertical, symbol Connector:Conn_01x04_Male
- added J?: left wheel sensor, Connector_PinHeader_2.54mm:PinHeader_1x04_P2.54mm_Vertical, symbol Connector:Conn_01x04_Male
- added J?: Phototransistor, Connector_PinHeader_2.54mm:PinHeader_1x02_P2.54mm_Vertical, symbol Connector:Conn_01x02_Male
- added J?: Analogue inputs, Connector_PinHeader_2.54mm:PinHeader_1x03_P2.54mm_Vertical, symbol Connector:Conn_01x03_Male
- added J?: right wheel sensor, Connector_PinHeader_2.54mm:PinHeader_1x04_P2.54mm_Vertical, symbol Connector:Conn_01x04_Male
- added J?: USB-to-controller, Connector_USB:USB_Micro-B_Wuerth_629105150521, symbol Connector:USB_OTG
- added J?: USB-from-battery, Connector_USB:USB_Micro-B_Wuerth_629105150521, symbol Connector:USB_OTG
- added J?: power switch, Connector_PinHeader_2.54mm:PinHeader_1x02_P2.54mm_Vertical, symbol Connector:Conn_01x02_Male
- added J?: power-connector, Connector_PinHeader_2.54mm:PinHeader_1x03_P2.54mm_Vertical, symbol Connector:Conn_01x03_Male
- added J?: data-connector, Connector_PinHeader_2.54mm:PinHeader_1x03_P2.54mm_Vertical, symbol Connector:Conn_01x03_Male
- added JP?: 0x48, Jumper:SolderJumper-2_P1.3mm_Open_RoundedPad1.0x1.5mm, symbol Device:Jumper_NO_Small
- added JP?: 0x49, Jumper:SolderJumper-2_P1.3mm_Open_RoundedPad1.0x1.5mm, symbol Device:Jumper_NO_Small
- added JP?: 0x4A, Jumper:SolderJumper-2_P1.3mm_Open_RoundedPad1.0x1.5mm, symbol Device:Jumper_NO_Small
- added JP?: 0x4B, Jumper:SolderJumper-2_P1.3mm_Open_RoundedPad1.0x1.5mm, symbol Device:Jumper_NO_Small
- added JP?: l->a2, Jumper:SolderJumper-2_P1.3mm_Open_RoundedPad1.0x1.5mm, symbol Device:Jumper_NO_Small
- added JP?: r->a3, Jumper:SolderJumper-2_P1.3mm_Open_RoundedPad1.0x1.5mm, symbol Device:Jumper_NO_Small
- added R? (x2): 220R, Resistor_SMD:R_0805_2012Metric, symbol Device:R_Small
- added R? (x3): 10K, Resistor_SMD:R_0805_2012Metric, symbol Device:R_Small
- added R?: 6K8, Resistor_SMD:R_0805_2012Metric, symbol Device:R_Small
- added R?: 33K, Resistor_SMD:R_0805_2012Metric, symbol Device:R_Small
- added R? (x2): 15K, Resistor_SMD:R_0805_2012Metric, symbol Device:R_Small
- added U? (x3): LM2903, Package_SO:Diodes_SO-8EP, symbol Comparator:LM2903
- added U?: adafruit-1015, reprapltd-kicad:adafruit-1015, symbol reprapltd-kicad:adafruit-1015
- added U?: AP1117-33, Package_TO_SOT_SMD:SOT-223-3_TabPin2, symbol Regulator_Linear:AP1117-33
Connections:
- net +3V3: now also C?.1, C?.1, C?.1, C?.1, C?.1, J?.2 (Pin_2), J?.4 (Pin_4), JP?.2, R?.1, R?.1, R?.2, R?.2, R?.2, R?.2, U?.1 (Vdd), U?.2 (VO), U?.8 (V+)
- net +5V: now also C?.1, C?.1, J?.1 (Pin_1), J?.1 (VBUS), J?.3 (Pin_3), R?.1, U?.3 (VI)
- net GND: now also U1.7 (GND), C?.2, C?.2, C?.2, C?.2, C?.2, C?.2, C?.2, C?.2, J?.1 (Pin_1), J?.1 (Pin_1), J?.1 (Pin_1), J?.1 (Pin_1), J?.3 (Pin_3), J?.3 (Pin_3), J?.3 (Pin_3), J?.5 (GND), J?.5 (GND), J?.6 (Shield), J?.6 (Shield), JP?.2, R?.2, R?.2, U?.1 (GND), U?.2 (GND), U?.4 (V-)
- net SCL-GPIO3: now also J?.1 (Pin_1), J?.2 (Pin_2), JP?.2, U?.3 (SCL)
- net SDA-GPIO2: now also J?.2 (Pin_2), J?.3 (Pin_3), JP?.2, U?.4 (SDA)
- net GPIO12 renamed E1
- net GPIO13 renamed E4
- net GPIO16 renamed E2
- net GPIO6 renamed E3
- new net: J?.1 (Pin_1), R?.1 (x2)
- new net: JP?.1, JP?.1, JP?.1, JP?.1, U?.5 (ADDR)
- new net: J?.4 (Pin_4), JP?.1, R?.1, U?.3 (+)
- new net: J?.4 (Pin_4), JP?.1, R?.1, U?.5 (+)
- new net: R?.1, R?.2, U?.2 (-), U?.6 (_)
- new net: J?.3 (Pin_3), JP?.2, U?.10 (A3)
- new net: C?.1, R?.1, R?.2, U?.7 (A0)
- new net: J?.2 (Pin_2), R?.2, U?.8 (A1)
- new net: J?.2 (Pin_2), JP?.2, U?.9 (A2)
- new net: J?.2 (D-), J?.2 (D-)
- new net: J?.3 (D+), J?.3 (D+)
- new net: J?.4 (ID), J?.4 (ID)
- new net: J?.1 (VBUS), J?.2 (Pin_2)
- new net E5: J?.2 (Pin_2)
- new net E6: U?.1
- new net E7: J?.2 (Pin_2)
- new net E8: U?.7
Other:
- note added: "10mA"
- note added: "Opto diode 1.16V; min ~= 800, max ~= 900; 0.782, 0.879; 2.58, 2.9v; 0.5 ->0.83\nBattery connects to charge connector by its own USB"
- note added: "battery voltage"
- note removed: "Opto diode 1.16V"

Commit message: Frank 2.0 electronics WIP.
Parts:
- removed J?: data-connector, Connector_PinHeader_2.54mm:PinHeader_1x03_P2.54mm_Vertical, symbol Connector:Conn_01x03_Male
- removed JP?: 0x48, Jumper:SolderJumper-2_P1.3mm_Open_RoundedPad1.0x1.5mm, symbol Device:Jumper_NO_Small
- removed JP?: 0x49, Jumper:SolderJumper-2_P1.3mm_Open_RoundedPad1.0x1.5mm, symbol Device:Jumper_NO_Small
- removed JP?: 0x4A, Jumper:SolderJumper-2_P1.3mm_Open_RoundedPad1.0x1.5mm, symbol Device:Jumper_NO_Small
- removed JP?: 0x4B, Jumper:SolderJumper-2_P1.3mm_Open_RoundedPad1.0x1.5mm, symbol Device:Jumper_NO_Small
- added C11, C12: 0.1u, Capacitor_SMD:C_0805_2012Metric, symbol Device:C_Small
- added J12: servo 3, Connector_PinHeader_2.54mm:PinHeader_1x03_P2.54mm_Vertical, symbol Connector:Conn_01x03_Male
- added J13: servo 2, Connector_PinHeader_2.54mm:PinHeader_1x03_P2.54mm_Vertical, symbol Connector:Conn_01x03_Male
- added J14: servo 1, Connector_PinHeader_2.54mm:PinHeader_1x03_P2.54mm_Vertical, symbol Connector:Conn_01x03_Male
- added J15: GPIO, Connector_PinHeader_2.54mm:PinHeader_1x05_P2.54mm_Vertical, symbol Connector:Conn_01x05_Male
- added J16: data-connector, Connector_PinHeader_2.54mm:PinHeader_1x04_P2.54mm_Vertical, symbol Connector:Conn_01x04_Male
- added U5: sparkfun-sx1509, reprapltd-kicad:sparkfun-sx1509, symbol reprapltd-kicad:sparkfun-sx1509
- gave numbers to parts that had none: 31
Connections:
- net +3V3: now also C12.2, U5.13 (3V3), U5.22 (VC1), U5.5 (VC2)
- net +5V: now also J12.2 (Pin_2), J13.2 (Pin_2), J14.2 (Pin_2)
- net GND: now also U3.5 (ADDR), C11.2, C12.1, J12.1 (Pin_1), J13.1 (Pin_1), J14.1 (Pin_1), J15.5 (Pin_5), J16.1 (Pin_1), U5.10 (GND), U5.14 (GND), U5.17 (GND)
- net at R10.1, R9.2, U2.2 (-)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: now also C11.1
- net IO8: now reaches U3.6 (ALRT)
- net IO8: now also U5.1 (IO8)
- net E1 renamed IO3
- net IO3: now also U5.21 (IO3)
- net E2 renamed IO2
- net IO2: now also U5.20 (IO2)
- net E3 renamed IO1
- net IO1: now also U5.19 (IO1)
- net E4 renamed IO0
- net IO0: now also U5.18 (IO0)
- net E5 renamed IO4
- net IO4: now also U5.23 (IO4)
- net E6 renamed IO5
- net IO5: now also U5.24 (IO5)
- net E7 renamed IO6
- net IO6: now also U5.25 (IO6)
- net E8 renamed IO7
- net IO7: now also U5.26 (IO7)
- net SCL-GPIO3 renamed SCL
- net SCL: now also J16.2 (Pin_2), U5.11 (SCL)
- net SDA-GPIO2 renamed SDA
- net SDA: now also J16.3 (Pin_3), U5.12 (SDA)
- new net: J14.3 (Pin_3), U5.2 (IO9)
- new net: J13.3 (Pin_3), U5.3 (IO10)
- new net: J12.3 (Pin_3), U5.4 (IO11)
- new net: J15.1 (Pin_1), U5.6 (IO12)
- new net: J15.2 (Pin_2), U5.7 (IO13)
- new net: J15.3 (Pin_3), U5.8 (IO14)
- new net: J15.4 (Pin_4), U5.9 (IO15)
- new net INTERRUPT: J16.4 (Pin_4), U5.16 (INT)
Other:
- note added: "0x29"
- note added: "0x3E"
- note added: "0x48"
- moved on the sheet: C8, J7, R11, R12, R13

Commit message: Now with indicator LEDs...
Parts:
- removed J15: GPIO, Connector_PinHeader_2.54mm:PinHeader_1x05_P2.54mm_Vertical, symbol Connector:Conn_01x05_Male
- added D1: FLASH, LED_SMD:LED_0805_2012Metric, symbol Device:LED_Small
- added D2: 5VLED, LED_SMD:LED_0805_2012Metric, symbol Device:LED_Small
- added D3: 3V3LED, LED_SMD:LED_0805_2012Metric, symbol Device:LED_Small
- added J15: GPIO, Connector_PinHeader_2.54mm:PinHeader_1x04_P2.54mm_Vertical, symbol Connector:Conn_01x04_Male
- added R14, R15, R16: 220R, Resistor_SMD:R_0805_2012Metric, symbol Device:R_Small
Connections:
- net +3V3: now also R14.1, R16.2
- net +5V: now also R15.2
- net GND: now also D2.1 (K), D3.1 (K), J15.4 (Pin_4)
- net at U5.6 (IO12): now also D1.1 (K)
- net at U5.7 (IO13): now also J15.1 (Pin_1)
- net at U5.8 (IO14): now also J15.2 (Pin_2)
- net at U5.9 (IO15): now also J15.3 (Pin_3)
- new net: D3.2 (A), R16.1
- new net: D2.2 (A), R15.1
- new net: D1.2 (A), R14.2
Other:
- moved on the sheet: J11
Changed lines of the file:
@@
 L Connector:Conn_01x03_Male J11
 U 1 1 5F0CD551
-P 10925 2100
-F 0 "J11" V 10987 2244 50  0000 L CNN
-F 1 "power-connector" V 10850 1850 50  0000 L CNN
-F 2 "Connector_PinHeader_2.54mm:PinHeader_1x03_P2.54mm_Vertical" H 10925 2100 50  0001 C CNN
-F 3 "~" H 10925 2100 50  0001 C CNN
-	1    10925 2100
+P 10950 3700
+F 0 "J11" V 11012 3844 50  0000 L CNN
+F 1 "power-connector" V 10875 3450 50  0000 L CNN
+F 2 "Connector_PinHeader_2.54mm:PinHeader_1x03_P2.54mm_Vertical" H 10950 3700 50  0001 C CNN
+F 3 "~" H 10950 3700 50  0001 C CNN
+	1    10950 3700
 	-1   0    0    1
 $EndComp
@@
 L power:+5V #PWR0135
 U 1 1 5F0CF071
-P 10650 1950
-F 0 "#PWR0135" H 10650 1800 50  0001 C CNN
-F 1 "+5V" H 10665 2123 50  0000 C CNN
-F 2 "" H 10650 1950 50  0001 C CNN
-F 3 "" H 10650 1950 50  0001 C CNN
-	1    10650 1950
+P 10675 3550
+F 0 "#PWR0135" H 10675 3400 50  0001 C CNN
+F 1 "+5V" H 10690 3723 50  0000 C CNN
+F 2 "" H 10675 3550 50  0001 C CNN
+F 3 "" H 10675 3550 50  0001 C CNN
+	1    10675 3550
 	1    0    0    -1
 $EndComp
@@
 L power:+3.3V #PWR0136
 U 1 1 5F0CF608
-P 10450 1950
-F 0 "#PWR0136" H 10450 1800 50  0001 C CNN
-F 1 "+3.3V" H 10465 2123 50  0000 C CNN
-F 2 "" H 10450 1950 50  0001 C CNN
-F 3 "" H 10450 1950 50  0001 C CNN
-	1    10450 1950
+P 10475 3550
+F 0 "#PWR0136" H 10475 3400 50  0001 C CNN
+F 1 "+3.3V" H 10490 3723 50  0000 C CNN
+F 2 "" H 10475 3550 50  0001 C CNN
+F 3 "" H 10475 3550 50  0001 C CNN
+	1    10475 3550
 	1    0    0    -1
 $EndComp
@@
 L power:GND #PWR0137
 U 1 1 5F0CFC12
-P 10650 2250
-F 0 "#PWR0137" H 10650 2000 50  0001 C CNN
-F 1 "GND" H 10655 2077 50  0000 C CNN
-F 2 "" H 10650 2250 50  0001 C CNN
-F 3 "" H 10650 2250 50  0001 C CNN
-	1    10650 2250
-	1    0    0    -1
-$EndComp
-Wire Wire Line
-	10725 2200 10650 2200
-Wire Wire Line
-	10650 2200 10650 2250
-Wire Wire Line
-	10725 2100 10450 2100
-Wire Wire Line
-	10450 2100 10450 1950
-Wire Wire Line
-	10725 2000 10650 2000
-Wire Wire Line
-	10650 2000 10650 1950
+P 10675 3850
+F 0 "#PWR0137" H 10675 3600 50  0001 C CNN
+F 1 "GND" H 10680 3677 50  0000 C CNN
+F 2 "" H 10675 3850 50  0001 C CNN
+F 3 "" H 10675 3850 50  0001 C CNN
+	1    10675 3850
+	1    0    0    -1
+$EndComp
+Wire Wire Line
+	10750 3800 10675 3800
+Wire Wire Line
+	10675 3800 10675 3850
+Wire Wire Line
+	10750 3700 10475 3700
+Wire Wire Line
+	10750 3600 10675 3600
+Wire Wire Line
+	10675 3600 10675 3550
 $Comp
 L power:GND #PWR0138
@@
 	5850 2925 5850 2800
 Connection ~ 5450 2925
-$Comp
-L Connector:Conn_01x05_Male J15
-U 1 1 5F116CDD
-P 5950 3675
-F 0 "J15" H 6000 3400 50  0000 C CNN
-F 1 "GPIO" V 5875 3675 50  0000 C CNN
-F 2 "Connector_PinHeader_2.54mm:PinHeader_1x05_P2.54mm_Vertical" H 5950 3675 50  0001 C CNN
-F 3 "~" H 5950 3675 50  0001 C CNN
-	1    5950 3675
-	1    0    0    -1
-$EndComp
-Wire Wire Line
-	6150 3475 6425 3475
 Wire Wire Line
 	6150 3575 6425 3575
@@
 	6575 5000 6575 4875
 Connection ~ 6775 5000
+$Comp
+L Device:R_Small R16
+U 1 1 5EC9242B
+P 10375 3700
+F 0 "R16" V 10179 3700 50  0000 C CNN
+F 1 "220R" V 10270 3700 50  0000 C CNN
+F 2 "Resistor_SMD:R_0805_2012Metric" H 10375 3700 50  0001 C CNN
+F 3 "~" H 10375 3700 50  0001 C CNN
+	1    10375 3700
+	0    -1   -1   0
+$EndComp
+$Comp
+L Device:R_Small R15
+U 1 1 5EC93474
+P 10125 3600
+F 0 "R15" V 10275 3600 50  0000 C CNN
+F 1 "220R" V 10200 3600 50  0000 C CNN
+F 2 "Resistor_SMD:R_0805_2012Metric" H 10125 3600 50  0001 C CNN
+F 3 "~" H 10125 3600 50  0001 C CNN
+	1    10125 3600
+	0    -1   -1   0
+$EndComp
+Connection ~ 10475 3700
+Wire Wire Line
+	10475 3550 10475 3700
+Wire Wire Line
+	10675 3600 10225 3600
+Connection ~ 10675 3600
+Wire Wire Line
+	10025 3600 9875 3600
+Wire Wire Line
+	10275 3700 10200 3700
+Wire Wire Line
+	10200 3700 10200 3800
+Wire Wire Line
+	10200 3800 9875 3800
+$Comp
+L power:GND #PWR0145
+U 1 1 5ED22480
+P 9575 3925
+F 0 "#PWR0145" H 9575 3675 50  0001 C CNN
+F 1 "GND" H 9580 3752 50  0000 C CNN
+F 2 "" H 9575 3925 50  0001 C CNN
+F 3 "" H 9575 3925 50  0001 C CNN
+	1    9575 3925
+	1    0    0    -1
+$EndComp
+$Comp
+L Connector:Conn_01x04_Male J15
+U 1 1 5ED486D7
+P 5950 3675
+F 0 "J15" V 6012 3819 50  0000 L CNN
+F 1 "GPIO" V 5875 3500 50  0000 L CNN
+F 2 "Connector_PinHeader_2.54mm:PinHeader_1x04_P2.54mm_Vertical" H 5950 3675 50  0001 C CNN
+F 3 "~" H 5950 3675 50  0001 C CNN
+	1    5950 3675
+	1    0    0    -1
+$EndComp
+$Comp
+L Device:R_Small R14
+U 1 1 5ED6E2BB
+P 5350 3475
+F 0 "R14" V 5154 3475 50  0000 C CNN
+F 1 "220R" V 5245 3475 50  0000 C CNN
+F 2 "Resistor_SMD:R_0805_2012Metric" H 5350 3475 50  0001 C CNN
+F 3 "~" H 5350 3475 50  0001 C CNN
+	1    5350 3475
+	0    -1   -1   0
+$EndComp
+$Comp
+L power:+3.3V #PWR0146
+U 1 1 5ED82DCA
+P 5150 3475
+F 0 "#PWR0146" H 5150 3325 50  0001 C CNN
+F 1 "+3.3V" H 5000 3550 50  0000 C CNN
+F 2 "" H 5150 3475 50  0001 C CNN
+F 3 "" H 5150 3475 50  0001 C CNN
+	1    5150 3475
+	1    0    0    -1
+$EndComp
+Wire Wire Line
+	5250 3475 5150 3475
+$Comp
+L Device:LED_Small D1
+U 1 1 5EDA984E
+P 5700 3475
+F 0 "D1" H 5700 3268 50  0000 C CNN
+F 1 "FLASH" H 5700 3359 50  0000 C CNN
+F 2 "LED_SMD:LED_0805_2012Metric" V 5700 3475 50  0001 C CNN
+F 3 "~" V 5700 3475 50  0001 C CNN
+	1    5700 3475
+	-1   0    0    1
+$EndComp
+Wire Wire Line
+	5800 3475 6425 3475
+Wire Wire Line
+	5450 3475 5600 3475
+$Comp
+L Device:LED_Small D2
+U 1 1 5EDD6E16
+P 9775 3600
+F 0 "D2" H 9775 3835 50  0000 C CNN
+F 1 "5VLED" H 9775 3744 50  0000 C CNN
+F 2 "LED_SMD:LED_0805_2012Metric" V 9775 3600 50  0001 C CNN
+F 3 "~" V 9775 3600 50  0001 C CNN
+	1    9775 3600
+	1    0    0    -1
+$EndComp
+Wire Wire Line
+	9575 3600 9575 3800
+$Comp
+L Device:LED_Small D3
+U 1 1 5EDDE768
+P 9775 3800
+F 0 "D3" H 9775 4035 50  0000 C CNN
+F 1 "3V3LED" H 9775 3944 50  0000 C CNN
+F 2 "LED_SMD:LED_0805_2012Metric" V 9775 3800 50  0001 C CNN
+F 3 "~" V 9775 3800 50  0001 C CNN
+	1    9775 3800
+	1    0    0    -1
+$EndComp
+Wire Wire Line
+	9675 3600 9575 3600
+Wire Wire Line
+	9675 3800 9575 3800
+Connection ~ 9575 3800
+Wire Wire Line
+	9575 3800 9575 3925
 $EndSCHEMATC

Commit message: Electronics WIP
Parts:
- added C13, C14: 0.1u, Capacitor_SMD:C_0805_2012Metric, symbol Device:C_Small
- D1, D2, D3: footprint LED_SMD:LED_0805_2012Metric -> LED_THT:LED_D3.0mm
Connections:
- net +3V3: now also C14.1
- net +5V: now also C13.1
- net GND: now also C13.2, C14.2
- net IO0: now also U1.12 (PWMB); no longer U1.18 (PWMA)
- net IO1: now also R3.2, U1.14 (BIN1); no longer R4.2, U1.16 (AIN1)
- net IO2: now also R4.2, U1.16 (AIN1); no longer R3.2, U1.14 (BIN1)
- net IO3: now also U1.18 (PWMA); no longer U1.12 (PWMB)
Other:
- moved on the sheet: C10, C9, J10, J8, J9, U4

Commit message: PCB WIP
Parts:
- added H1, H2, H3, H4: MountingHole, MountingHole:MountingHole_3.2mm_M3, symbol Mechanical:MountingHole
- U2: footprint Package_SO:Diodes_SO-8EP -> reprapltd-kicad:Diodes_SO-8EP
Connections:
- net IO0: now also J1.2 (Pin_2); no longer U1.12 (PWMB)
- net IO1: now also U2.1; no longer R3.2, U1.14 (BIN1)
- net IO2: now also J4.2 (Pin_2); no longer R4.2, U1.16 (AIN1)
- net IO3: now also U2.7; no longer U1.18 (PWMA)
- net IO4: now also U1.12 (PWMB); no longer J1.2 (Pin_2)
- net IO5: now also R3.2, U1.14 (BIN1); no longer U2.1
- net IO6: now also R4.2, U1.16 (AIN1); no longer J4.2 (Pin_2)
- net IO7: now also U1.18 (PWMA); no longer U2.7
Changed lines of the file:
@@
 Connection ~ 2525 1500
 Text GLabel 2325 4225 3    50   Input ~ 0
-IO0
+IO4
 Text GLabel 2925 4225 3    50   Input ~ 0
-IO3
+IO7
 Text GLabel 2525 4225 3    50   Input ~ 0
-IO1
+IO5
 Text GLabel 2725 4225 3    50   Input ~ 0
-IO2
+IO6
 $Comp
 L Transistor_FET:DMN6075S Q1
@@
 $EndComp
 Text GLabel 1375 4925 2    50   Input ~ 0
-IO4
+IO0
 $Comp
 L power:GND #PWR0107
@@
 $EndComp
 Text GLabel 1325 6400 2    50   Input ~ 0
-IO6
+IO2
 $Comp
 L power:GND #PWR0111
@@
 F 0 "U2" H 2850 7217 50  0000 C CNN
 F 1 "LM2903" H 2850 7126 50  0000 C CNN
-F 2 "Package_SO:Diodes_SO-8EP" H 2850 6850 50  0001 C CNN
+F 2 "reprapltd-kicad:Diodes_SO-8EP" H 2850 6850 50  0001 C CNN
 F 3 "http://www.ti.com/lit/ds/symlink/lm393.pdf" H 2850 6850 50  0001 C CNN
 	2    2850 6850
@@
 F 0 "U2" H 2825 5742 50  0000 C CNN
 F 1 "LM2903" H 2825 5651 50  0000 C CNN
-F 2 "Package_SO:Diodes_SO-8EP" H 2825 5375 50  0001 C CNN
+F 2 "reprapltd-kicad:Diodes_SO-8EP" H 2825 5375 50  0001 C CNN
 F 3 "http://www.ti.com/lit/ds/symlink/lm393.pdf" H 2825 5375 50  0001 C CNN
 	1    2825 5375
@@
 	2175 5950 2175 6000
 Text GLabel 3250 5375 2    50   Input ~ 0
-IO5
+IO1
 Text GLabel 3275 6850 2    50   Input ~ 0
-IO7
+IO3
 Wire Wire Line
 	3125 5375 3250 5375
@@
 F 0 "U2" H 3183 6096 50  0000 L CNN
 F 1 "LM2903" H 3183 6005 50  0000 L CNN
-F 2 "Package_SO:Diodes_SO-8EP" H 3225 6050 50  0001 C CNN
+F 2 "reprapltd-kicad:Diodes_SO-8EP" H 3225 6050 50  0001 C CNN
 F 3 "http://www.ti.com/lit/ds/symlink/lm393.pdf" H 3225 6050 50  0001 C CNN
 	3    3225 6050
@@
 	10575 1450 10250 1450
 Connection ~ 10250 1450
+$Comp
+L Mechanical:MountingHole H1
+U 1 1 5ED741BD
+P 7850 5625
+F 0 "H1" H 7950 5671 50  0000 L CNN
+F 1 "MountingHole" H 7950 5580 50  0000 L CNN
+F 2 "MountingHole:MountingHole_3.2mm_M3" H 7850 5625 50  0001 C CNN
+F 3 "~" H 7850 5625 50  0001 C CNN
+	1    7850 5625
+	1    0    0    -1
+$EndComp
+$Comp
+L Mechanical:MountingHole H3
+U 1 1 5ED77C3D
+P 8200 5625
+F 0 "H3" H 8300 5671 50  0000 L CNN
+F 1 "MountingHole" H 8300 5580 50  0000 L CNN
+F 2 "MountingHole:MountingHole_3.2mm_M3" H 8200 5625 50  0001 C CNN
+F 3 "~" H 8200 5625 50  0001 C CNN
+	1    8200 5625
+	1    0    0    -1
+$EndComp
+$Comp
+L Mechanical:MountingHole H2
+U 1 1 5ED7858B
+P 7850 5850
+F 0 "H2" H 7950 5896 50  0000 L CNN
+F 1 "MountingHole" H 7950 5805 50  0000 L CNN
+F 2 "MountingHole:MountingHole_3.2mm_M3" H 7850 5850 50  0001 C CNN
+F 3 "~" H 7850 5850 50  0001 C CNN
+	1    7850 5850
+	1    0    0    -1
+$EndComp
+$Comp
+L Mechanical:MountingHole H4
+U 1 1 5ED78FCD
+P 8200 5850
+F 0 "H4" H 8300 5896 50  0000 L CNN
+F 1 "MountingHole" H 8300 5805 50  0000 L CNN
+F 2 "MountingHole:MountingHole_3.2mm_M3" H 8200 5850 50  0001 C CNN
+F 3 "~" H 8200 5850 50  0001 C CNN
+	1    8200 5850
+	1    0    0    -1
+$EndComp
 $EndSCHEMATC
