File: Frank 2.0/Electronics/Frank-2-Pi/Frank-2-Pi.sch (KiCad schematic (older format))
At the start: 64 parts, among them J1 left wheel sensor, J10 USB-to-controller, J11 power-connector, J12 servo 3, J13 servo 2, J14 servo 1, J15 GPIO, J16 data-connector, J2 Left motor, J3 Right motor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

Commit message: Updating
Parts:
- J10, J8: symbol Connector:USB_OTG -> Frank-2-Pi-rescue:USB_OTG-Connector
Changed lines of the file:
@@
 	10250 1000 10400 1000
 $Comp
-L Connector:USB_OTG J10
+L Frank-2-Pi-rescue:USB_OTG-Connector J10
 U 1 1 5EF4CF78
 P 8400 1200
@@
 	8400 1600 8400 1675
 $Comp
-L Connector:USB_OTG J8
+L Frank-2-Pi-rescue:USB_OTG-Connector J8
 U 1 1 5EFB8934
 P 6925 1200
